Commit message: PD Controller for joints added for Go1 Robot

File: robot/Go1.urdf (robot description, URDF)
Before this commit: robot go1, 38 links, 37 joints
Links:
- removed link camera_chin
- removed link camera_face
- removed link camera_laserscan_link_left
- removed link camera_laserscan_link_right
- removed link camera_left
- removed link camera_optical_chin
- removed link camera_optical_face
- removed link camera_optical_left
- removed link camera_optical_rearDown
- removed link camera_optical_right
- removed link camera_rearDown
- removed link camera_right
- removed link ultraSound_face
- removed link ultraSound_left
- removed link ultraSound_right
Joints:
- removed joint camera_joint_chin
- removed joint camera_joint_face
- removed joint camera_joint_left
- removed joint camera_joint_rearDown
- removed joint camera_joint_right
- removed joint camera_laserscan_joint_left
- removed joint camera_laserscan_joint_right
- removed joint camera_optical_joint_chin
- removed joint camera_optical_joint_face
- removed joint camera_optical_joint_left
- removed joint camera_optical_joint_rearDown
- removed joint camera_optical_joint_right
- removed joint ultraSound_joint_face
- removed joint ultraSound_joint_left
- removed joint ultraSound_joint_right
